File: pcb/FightKeySmol.kicad_pcb (KiCad board)
At the start: 2 copper layers, 254 x 85.1 mm, 31 parts, among them J1 Conn_01x08_Male, J2 Conn_01x08_Male, U1 Pico

Commit message: kicad_pcb: updated for schem and new tiny design
Signed-off-by: Dylan Turner <dylantdmt@gmail.com>
Parts:
- removed J1, J2: Conn_01x08_Male, Connector_PinHeader_2.54mm:PinHeader_1x08_P2.54mm_Vertical
- removed R_DOWN1, R_K1, R_K2, R_K3, R_K4, R_LEFT1, R_P1, R_P2, R_P3, R_P4, R_RIGHT1, R_SELECT1, R_START1, R_UP1: R, Resistor_THT:R_Axial_DIN0204_L3.6mm_D1.6mm_P2.54mm_Vertical
- U1: moved to B.Cu
- moved AK_BTN1 62.0 mm to (199.4, 114.3)
- moved AP_BT1 62.0 mm to (199.4, 75.6)
- moved MK_BTN1 62.0 mm to (155.6, 105.4)
- moved MP_BTN1 62.0 mm to (155.6, 66.7)
- moved HP_BTN1 62.0 mm to (177.8, 66.7)
- moved LP_BTN1 62.0 mm to (134.0, 84.5)
- moved HK_BTN1 62.0 mm to (177.8, 105.4)
- moved LK_BTN1 62.0 mm to (134.0, 123.2)
- moved U1 47.4 mm to (118.7, 76.8), turned to 180 degrees
- moved UP_BTN1 41.7 mm to (90.5, 79.7), turned to -30 degrees
- moved RIGHT_BTN1 34.6 mm to (98.4, 109.2), turned to -30 degrees
- moved DOWN_BTN1 30.7 mm to (79.7, 98.4), turned to -30 degrees
- moved LEFT_BTN1 30.7 mm to (61.0, 87.6), turned to -30 degrees
- moved START_BTN1 26.4 mm to (94.6, 58.4)
- moved SELECT_BTN1 24.3 mm to (71.8, 58.4)
Connections:
- AK_BTN1 pad 1: /VCC -> /GND
- AP_BT1 pad 1: /VCC -> /GND
- DOWN_BTN1 pad 1: /VCCL -> /GND
- DOWN_BTN1 pad 2: /DOWNL -> /DOWN
- HK_BTN1 pad 1: /VCC -> /GND
- HP_BTN1 pad 1: /VCC -> /GND
- LEFT_BTN1 pad 1: /VCCL -> /GND
- LEFT_BTN1 pad 2: /LEFTL -> /LEFT
- LK_BTN1 pad 1: /VCC -> /GND
- LP_BTN1 pad 1: /VCC -> /GND
- MK_BTN1 pad 1: /VCC -> /GND
- MP_BTN1 pad 1: /VCC -> /GND
- RIGHT_BTN1 pad 1: /VCCL -> /GND
- RIGHT_BTN1 pad 2: /RIGHTL -> /RIGHT
- SELECT_BTN1 pad 1: /VCCL -> /GND
- SELECT_BTN1 pad 2: /SELECTL -> /SELECT
- START_BTN1 pad 1: /VCCL -> /GND
- START_BTN1 pad 2: /STARTL -> /START
- U1 pad 10: /STARTR -> /MK
- U1 pad 11: /SELECTR -> /AK
- U1 pad 12: /LK -> /AP
- U1 pad 14: /MK -> /LP
- U1 pad 15: /HK -> /MP
- U1 pad 16: /AP -> /HK
- U1 pad 17: /LP -> /HP
- U1 pad 20: /HP -> unconnected-(U1-Pad20)
- U1 pad 21: /AK -> /START
- U1 pad 22: /MP -> /SELECT
- U1 pad 3: unconnected-(U1-Pad3) -> /GND
- U1 pad 36: /VCC -> unconnected-(U1-Pad36)
- U1 pad 4: /UPR -> /UP
- U1 pad 5: /DOWNR -> /DOWN
- U1 pad 6: /LEFTR -> /RIGHT
- U1 pad 7: /RIGHTR -> /LEFT
- U1 pad 9: unconnected-(U1-Pad9) -> /LK
- UP_BTN1 pad 1: /VCCL -> /GND
- UP_BTN1 pad 2: /UPL -> /UP
Routing:
- net /GNDL: track 308.2 -> 0.00 mm
- net /VCC: track 297.8 -> 0.00 mm, vias 1 -> 0
- net /VCCL: track 204.7 -> 0.00 mm
- net /LEFTL: track 114.7 -> 0.00 mm, vias 2 -> 0
- net /SELECTL: track 112.0 -> 0.00 mm, vias 1 -> 0
- net /DOWNL: track 111.9 -> 0.00 mm
- net /LEFT: track 0.00 -> 95.0 mm, vias 0 -> 1
- net /GND: track 291.4 -> 382.4 mm, vias 3 -> 0
- net /UPL: track 87.6 -> 0.00 mm
- net /STARTL: track 82.1 -> 0.00 mm
- net /DOWN: track 0.00 -> 72.5 mm
- net /LP: track 84.2 -> 14.8 mm, vias 2 -> 0
- net /RIGHTL: track 67.9 -> 0.00 mm
- net /RIGHTR: track 62.3 -> 0.00 mm
- net /LEFTR: track 61.9 -> 0.00 mm
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Other:
- board size 254 x 85.1 mm -> 168.9 x 83.8 mm
- board text added: "Created by Dylan Turner"
- board text added: "Fight Key Smol"
- board text removed: "Create by Dylan Turner"
